Commit message: Visual odometry with Gazebo (#88)
* First approach on visual odometry with Gazebo

* Fix for multiple robots

* Remove default position

* Allow disabling VO

* Change camera_height

* Add namespace

* Revert

* Move some scripts from ca_visual_odometry to ca_camera

* Move bringup of ca_visual_odometry from gazebo to navigation

* Some fixes to raspicam launch files

* Fix dependencies

* Make Hz test easy to pass

File: ca_description/urdf/sensors/camera_generic.xacro (robot description, xacro)
@@ -9,5 +9,5 @@
     <link name="${name}_link"/>
     <joint name="${name}_optical_joint" type="fixed">
-      <origin xyz="0 0 0" rpy="${-pi/2} 0 ${-pi/2}" />
+      <origin rpy="${-pi/2} 0 ${-pi/2}" />
       <parent link="${name}_link" />
       <child link="${name}_optical_frame"/>
